File: Design/Long ISP PCB/shem.brd (EAGLE design)
At the start: 132.3 x 78 mm, 41 parts, among them IC1 4511N, IC2 4511N, J1 9V_POWER_JACK, Q1 600mA/40V, Q2 600mA/40V, Q3 600mA/40V, Q4 600mA/40V, Q5 600mA/40V, U2 328P, U3 SN74HC595N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

Commit message: fixed board schematic consistency sync issue as a result leds for input switches have been removed again
Parts:
- removed D1, D2, D3, D4, D5, D6, D7, D8: (no value), SparkFun-LED:LED_3MM
- moved PWR 46.6 mm to (-11.4, 33.0)
- moved C1 26.8 mm to (-12.7, 40.6)
- moved C2 25.5 mm to (-12.7, 45.7)
- moved U1 15.5 mm to (2.54, 34.3)
- moved S8 13.0 mm to (-2.11, 8.24)
- moved S7 12.2 mm to (11.6, 8.24)
- moved IC1 11.4 mm to (20.3, 38.1)
- moved S1 11.4 mm to (101.7, 8.24)
- moved S6 10.6 mm to (26.3, 8.24)
- moved S2 9.22 mm to (87.3, 8.24)
- moved S5 8.60 mm to (42.0, 8.24)
- moved S3 7.28 mm to (71.8, 8.24)
- moved S4 7.07 mm to (57.4, 8.24)
- moved U3 5.08 mm to (92.7, 38.1)
- moved LS1 3.59 mm to (11.4, 54.6)
Connections:
- net 9V: now also J1.PWR; no longer IC1.16, IC1.3, IC1.4, IC2.16, IC2.3, IC2.4, PWR.P, PWR.S
- net N$1: now also C2.1, PWR.S, U1.OUT; no longer J1.PWR, PWR.O
- net VCC: now also IC1.16, IC1.3, IC1.4, IC2.16, IC2.3, IC2.4, PWR.P; no longer C2.1, U1.OUT
Routing:
- net GND: track 473.1 -> 0.00 mm, vias 2 -> 0
- net SCK: track 293.7 -> 0.00 mm, vias 4 -> 0
- net VCC: track 277.6 -> 0.00 mm, vias 3 -> 0
- net 9V: track 181.1 -> 0.00 mm
- net SCORE_TENS_ENABLE: track 148.0 -> 0.00 mm, vias 5 -> 0
- net MISO: track 134.9 -> 0.00 mm, vias 3 -> 0
- net MOSI: track 131.5 -> 0.00 mm, vias 5 -> 0
- net S1: track 128.5 -> 0.00 mm, vias 1 -> 0
- net S0: track 112.2 -> 0.00 mm, vias 1 -> 0
- net S2: track 111.4 -> 0.00 mm, vias 1 -> 0
- net BUZZ: track 108.9 -> 0.00 mm, vias 1 -> 0
- net IC: track 105.6 -> 0.00 mm, vias 4 -> 0
- net S3: track 97.4 -> 0.00 mm, vias 1 -> 0
- net S7: track 95.3 -> 0.00 mm
- net SCORE_ONES_ENABLE: track 84.0 -> 0.00 mm, vias 2 -> 0
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Other:
- board size 132.3 x 78 mm -> 132.3 x 72.8 mm

Commit message: re added led indicators to inputswitches
Parts:
- added D1, D2, D3, D4, D5, D6, D7, D8: (no value), SparkFun-LED:LED_3MM
- added R2, R3, R4, R5, R6, R7, R8, R9: 330, SparkFun-Resistors:AXIAL-0.3
Connections:
- new net N$12: D1.K, R2.P$2
- new net N$13: D8.K, R9.P$2
- new net N$14: D7.K, R8.P$2
- new net N$15: D6.K, R7.P$2
- new net N$17: D5.K, R6.P$2
- new net N$18: D4.K, R5.P$2
- new net N$19: D3.K, R4.P$2
- new net N$20: D2.K, R3.P$2
- net GND: now also R2.P$1, R3.P$1, R4.P$1, R5.P$1, R6.P$1, R7.P$1, R8.P$1, R9.P$1
- net S0: now also D1.A
- net S1: now also D2.A
- net S2: now also D3.A
- net S3: now also D4.A
- net S4: now also D5.A
- net S5: now also D6.A
- net S6: now also D7.A
- net S7: now also D8.A

Commit message: laid out new components and autorouted the board
Parts:
- moved R9 316.6 mm to (2.00, 18.0), turned to 90 degrees
- moved R8 298.9 mm to (16.0, 18.0), turned to 90 degrees
- moved R7 282.3 mm to (31.0, 18.0), turned to 90 degrees
- moved R6 267.0 mm to (47.0, 18.0), turned to 90 degrees
- moved R5 253.0 mm to (62.0, 18.0), turned to 90 degrees
- moved D8 224.8 mm to (-2.00, 21.0), turned to 90 degrees
- moved D7 207.6 mm to (12.0, 21.0), turned to 90 degrees
- moved D6 191.8 mm to (26.0, 21.0), turned to 90 degrees
- moved D5 178.5 mm to (42.0, 21.0), turned to 90 degrees
- moved D4 167.3 mm to (57.0, 21.0), turned to 90 degrees
- moved D3 159.0 mm to (72.0, 21.0), turned to 90 degrees
- moved R4 143.1 mm to (77.0, 18.0), turned to 90 degrees
- moved D2 141.2 mm to (87.0, 21.0), turned to 90 degrees
- moved D1 133.9 mm to (102.0, 21.0), turned to 90 degrees
- moved R3 129.8 mm to (92.0, 18.0), turned to 90 degrees
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Routing:
- net GND: track 0.00 -> 529.0 mm, vias 0 -> 3
- net VCC: track 0.00 -> 342.2 mm, vias 0 -> 3
- net SCORE_TENS_ENABLE: track 0.00 -> 217.9 mm, vias 0 -> 2
- net MOSI: track 0.00 -> 216.8 mm, vias 0 -> 6
- net S0: track 0.00 -> 147.3 mm, vias 0 -> 3
- net S5: track 0.00 -> 142.3 mm, vias 0 -> 2
- net S3: track 0.00 -> 126.7 mm, vias 0 -> 3
- net SCK: track 0.00 -> 123.5 mm, vias 0 -> 2
- net MISO: track 0.00 -> 116.0 mm, vias 0 -> 3
- net S1: track 0.00 -> 114.3 mm, vias 0 -> 4
- net BUZZ: track 0.00 -> 113.1 mm, vias 0 -> 2
- net S7: track 0.00 -> 102.5 mm, vias 0 -> 3
- net S2: track 0.00 -> 96.8 mm, vias 0 -> 4
- net IC: track 0.00 -> 93.8 mm, vias 0 -> 3
- net S6: track 0.00 -> 89.6 mm, vias 0 -> 2
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